File: figtree.kicad_sch (KiCad schematic)
At the start: 18 parts, among them J1 USB_B_Micro, J2 CHG, J3 Off, J4 Batt, J5 OUT, Q1 SI2307, U1 TP4054, U2 BUCKBOOST, U3 ME6211

Commit message: Update png and pdfs
Parts:
- U2: value BUCKBOOST -> MOUNTING_FOOTPRINT
Changed lines of the file:
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@@
 (kicad_sch
-	(version 20231120)
+	(version 20250114)
 	(generator "eeschema")
-	(generator_version "8.0")
+	(generator_version "9.0")
 	(paper "A4")
 	(title_block
@@
 	(label "VIN"
 		(at 91.44 29.21 0)
-		(fields_autoplaced yes)
 		(effects
 			(font
@@
 	(label "CHRG"
 		(at 104.14 134.62 0)
-		(fields_autoplaced yes)
 		(effects
 			(font
@@
 	(label "D3+"
 		(at 102.87 119.38 90)
-		(fields_autoplaced yes)
 		(effects
 			(font
@@
 	(label "VOUT"
 		(at 207.01 22.86 0)
-		(fields_autoplaced yes)
 		(effects
 			(font
@@
 	(label "PROG"
 		(at 138.43 134.62 0)
-		(fields_autoplaced yes)
 		(effects
 			(font
@@
 	(label "CE"
 		(at 173.99 83.82 0)
-		(fields_autoplaced yes)
 		(effects
 			(font
@@
 		(shape input)
 		(at 204.47 50.8 0)
-		(fields_autoplaced yes)
 		(effects
 			(font
@@
 		(shape input)
 		(at 157.48 73.66 90)
-		(fields_autoplaced yes)
 		(effects
 			(font
@@
 			)
 		)
-		(property "Value" "BUCKBOOST"
+		(property "Value" "MOUNTING_FOOTPRINT"
 			(at 140.335 22.86 0)
 			(effects
@@
 		)
 	)
+	(embedded_fonts no)
 )
